File: Circuit/Circuit.kicad_sch (KiCad schematic)
At the start: 12 parts, among them SW1 SW_MEC_5G, SW2 SW_DPDT_x2, U1 LM317_TO-220

Commit message: finsihed PCB layout
Parts:
- removed ESP8266-01: PinHeader-2x4, Connector_PinHeader_2.54mm:PinHeader_2x04_P2.54mm_Vertical, symbol Connector_Generic:Conn_02x04_Counter_Clockwise
- removed SW1: SW_MEC_5G, Button_Switch_THT:SW_PUSH_6mm, symbol Switch:SW_MEC_5G
- added ESP8266: PinHeader_2x4, Connector_PinSocket_2.54mm:PinSocket_2x04_P2.54mm_Vertical, symbol Connector_Generic:Conn_02x04_Odd_Even
- added PowerIN1, Serial1: JST-2P, Connector_JST:JST_EH_B2B-EH-A_1x02_P2.50mm_Vertical, symbol Connector_Generic:Conn_01x02
- added SW1: SW_MEC_5E, Button_Switch_THT:SW_PUSH_6mm, symbol Switch:SW_MEC_5E
Connections:
- net +3.3V: now also ESP8266.2 (Pin_2)
- net GND: now also ESP8266.7 (Pin_7), PowerIN1.1 (Pin_1), SW1.1
- net RX: now also Serial1.2 (Pin_2)
- net TX: now also ESP8266.1 (Pin_1), Serial1.1 (Pin_1)
- net VCC: now also PowerIN1.2 (Pin_2)
- net at R5.2: now also ESP8266.3 (Pin_3)
- net at R3.2, R4.1: now also ESP8266.8 (Pin_8)
- net at SW2.2 (B): now also ESP8266.6 (Pin_6)
- new net: ESP8266.5 (Pin_5), SW1.2
Other:
- moved on the sheet: R1, R2, U1
